File: Synkino_KiCAD/gitfup.kicad_pcb (KiCad board)
At the start: 2 copper layers, 88.4 x 82.3 mm, 182 parts, among them J1 Pwr, J10 EYE8_OUT, J11 EYE4_OUT, J12 2.5mm, J13 EYE5_OUT, J2 2.5mm, J3 3.5mm, J4 Micro_SD_Card_Det_Hirose_DM3AT, J5 EYE1_OUT, J6 EYE6_OUT, J7 EYE2_OUT, J8 EYE7_OUT, J9 EYE3_OUT, Q1 IRF7319, Q2 BC847, Q3 IRLML2244, SW1 SW_Push, SW2 Rotary_Encoder_Switch, SW3 SW_Push, U1 MCP1702T-5002E/MB, U10 ATMEGA328P-AU, U11 QRE1113, U12 QRE1113, U13 QRE1113, U14 QRE1113, U15 QRE1113, U16 QRE1113, U18 QRE1113, U2 ATMEGA328P-AU, U3 74HC4050, U4 SPIOLED128x64, U5 AP7312-1833W6-7, U6 74HC14, U7 VS1053B, U8 MAX4741, U9 QRE1113, X1 FTDIconn, X2 ICSP, X3 FTDIconn, X4 ICSP, Y1 16Mhz, Y2 12.288MHz, Y3 16Mhz

Commit message: Versuchen, den HEAD zu retten
Parts:
- removed D6: BZX84C9V1, lib_fp:D_SOT-23_1A3K
- removed the GND at (125.2, 104.9)
- added D7: BZX84C9V1, lib_fp:D_SOT-23_1A3K, F.Cu at (101.6, 87.5)
- D4: value BZX84C9V1 -> AD4
- Q3: footprint TO_SOT_Packages_SMD:SOT-23_Handsoldering -> TO_SOT_Packages_SMD:SOT-23
- R30: value 470 -> 330
- moved R10 15.2 mm to (124.8, 104.3), turned to 180 degrees
- moved R9 14.6 mm to (125.1, 100.7)
- moved D3 12.2 mm to (74.9, 42.9)
- moved R49 6.83 mm to (106.3, 94.7)
- moved GND 6.35 mm to (74.9, 101.5)
- moved D1 5.51 mm to (105.7, 87.5), turned to 90 degrees
- moved C10 5.21 mm to (125.6, 86.4)
- moved   4.95 mm to (70.5, 103.6)
- moved   4.95 mm to (70.5, 41.9)
- moved X1 4.83 mm to (70.4, 85.1)
- moved SW1 4.49 mm to (109.7, 92.0)
- moved A0 3.81 mm to (70.4, 49.5)
- moved A1 3.81 mm to (70.4, 52.1)
- moved A2 3.81 mm to (70.4, 54.6)
- moved A3 3.81 mm to (70.4, 57.1)
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Connections:
- D4 pad 1: Net-(C2-Pad1) -> Net-(AD4-Pad1)
Routing:
- net Net-(AD4-Pad1): track 1.05 -> 24.2 mm, vias 0 -> 1
- net GND: track 210.4 -> 189.1 mm, vias 51 -> 46
- net Net-(C2-Pad1): track 68.6 -> 47.6 mm, vias 1 -> 0
- net Net-(C9-Pad2): track 33.0 -> 16.6 mm, vias 2 -> 0
- net /MISO_3V: track 91.1 -> 78.7 mm, vias 9 -> 8
- net Net-(D3-Pad2): track 46.9 -> 58.9 mm
- net /~PWR_OFF: track 60.4 -> 70.7 mm, vias 6 -> 5
- net Net-(C3-Pad2): track 71.0 -> 76.8 mm, vias 4 -> 6
- net +3V3: track 219.3 -> 224.8 mm
- net Net-(C4-Pad2): track 67.7 -> 72.6 mm
- net /CTRL_TXD: track 45.8 -> 50.6 mm
- net /CTRL_RXD: track 40.6 -> 45.4 mm
- net Net-(CD5-Pad1): track 27.0 -> 30.8 mm
- net Net-(CA3-Pad1): track 27.5 -> 31.3 mm
- net Net-(CA2-Pad1): track 24.5 -> 28.3 mm
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Other:
- board size 88.4 x 82.3 mm -> 93.3 x 82.3 mm
- board text added: "FTDI-A"
- board text added: "FTDI-C"
- board text added: "SCL"
- board text added: "SDA"
- board text added: "Synkino • Rev. B"
- board text removed: "MISO"
- board text removed: "Rev. B"
