File: Synkino_KiCAD/_autosave-Synkino.kicad_pcb (KiCad board)
At the start: 2 copper layers, 93.3 x 82.3 mm, 181 parts, among them J1 Pwr, J10 EYE8_OUT, J11 EYE4_OUT, J12 2.5mm, J13 EYE5_OUT, J2 2.5mm, J3 3.5mm, J4 Micro_SD_Card_Det_Hirose_DM3AT, J5 EYE1_OUT, J6 EYE6_OUT, J7 EYE2_OUT, J8 EYE7_OUT, J9 EYE3_OUT, Q1 IRF7319, Q2 BC847, Q3 IRLML2244, SW1 SW_Push, SW2 Rotary_Encoder_Switch, SW3 SW_Push, U1 MCP1702T-5002E/MB, U10 ATMEGA328P-AU, U11 QRE1113, U12 QRE1113, U13 QRE1113, U14 QRE1113, U15 QRE1113, U16 QRE1113, U18 QRE1113, U2 ATMEGA328P-AU, U3 74HC4050, U4 SPIOLED128x64, U5 AP7312-1833W6-7, U6 74HC14, U7 VS1053B, U8 MAX4741, U9 QRE1113, X1 FTDIconn, X2 ICSP, X3 FTDIconn, X4 ICSP, Y1 16Mhz, Y2 12.288MHz, Y3 16Mhz

Commit message: gerber cleanup
Parts:
- removed D5: CD5, Measurement_Points:Measurement_Point_Round-TH_Small
- removed the GND at (142.0, 101.6)
- added  : MountingHole_3.2mm_M3_DIN965, Mounting_Holes:MountingHole_3.2mm_M3_DIN965, F.Cu at (111.0, 103.6)
- added 3V3: 3V3, Measurement_Points:Measurement_Point_Round-TH_Small, F.Cu at (86.2, 46.1)
- added 5V: 5V, Measurement_Points:Measurement_Point_Round-TH_Small, F.Cu at (86.1, 41.7)
- added BZ1: Buzzer, lib_fp:AAC801J-13, F.Cu at (78.2, 89.7)
- added R51: 100, Resistors_SMD:R_0805_HandSoldering, F.Cu at (88.9, 80.8)
- added R53: 10k, Resistors_SMD:R_0805_HandSoldering, F.Cu at (105.4, 63.6)
- added U17: 24LC256, Housings_SOIC:SOIC-8_3.9x4.9mm_Pitch1.27mm, F.Cu at (78.2, 99.3)
- J3: footprint lib_fp:SJ1-352XNG -> lib_fp:SJ1-352XNG-3pin
- R30: value 330 -> 680
- R47: value 270 -> 680
- U4: footprint Synkino:SPIOLED -> lib_fp:SPIOLED
- X1, X3: footprint Pin_Headers:Pin_Header_Straight_1x06_Pitch2.54mm -> lib_fp:Pin_Header_Straight_1x06_Pitch2.54mm
- X2, X4: footprint Pin_Headers:Pin_Header_Straight_2x03_Pitch2.54mm -> lib_fp:Pin_Header_Straight_2x03_Pitch2.54mm
- moved GND 54.7 mm to (70.4, 47.0)
- moved X4 25.1 mm to (110.7, 93.2)
- moved R9 22.9 mm to (110.0, 83.6), turned to 90 degrees
- moved C3 18.0 mm to (136.7, 86.4), turned to 180 degrees
- moved C9 18.0 mm to (131.1, 86.4), turned to 180 degrees
- moved SW1 17.8 mm to (127.5, 92.0)
- moved U1 17.7 mm to (112.8, 97.8)
- moved R10 17.4 mm to (125.5, 86.9), turned to 270 degrees
- moved C10 17.4 mm to (123.7, 103.6), turned to 180 degrees
- moved C6 17.0 mm to (124.7, 99.6), turned to 270 degrees
- moved Q1 16.9 mm to (121.4, 92.2)
- moved C16 16.2 mm to (121.2, 99.6)
- moved R7 14.6 mm to (143.0, 86.6)
- moved X1 12.7 mm to (70.4, 97.8), turned to 180 degrees
- moved C2 12.3 mm to (118.4, 103.6)
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Connections:
- U2 pad 9: Net-(CD5-Pad1) -> /BUZZ
Routing:
- net +3V3: track 224.8 -> 284.0 mm, vias 8 -> 11
- net /SDA: track 67.0 -> 104.9 mm, vias 8 -> 10
- net /SCL: track 71.6 -> 108.3 mm, vias 2 -> 4
- net Net-(CD5-Pad1): track 30.8 -> 0.00 mm, vias 2 -> 0
- net Net-(C5-Pad2): track 48.8 -> 79.1 mm, vias 4 -> 3
- net /BUZZ: track 0.00 -> 28.5 mm, vias 0 -> 2
- net /MISO_3V: track 78.7 -> 104.8 mm, vias 8 -> 13
- net /MOSI_5V: track 42.0 -> 68.0 mm, vias 1 -> 3
- net /SCLK_5V: track 48.8 -> 72.2 mm, vias 2 -> 4
- net /OLED_RES: track 6.75 -> 29.7 mm, vias 1 -> 3
- net Net-(C5-Pad1): track 65.2 -> 42.8 mm
- net +5V: track 284.0 -> 306.0 mm, vias 15 -> 19
- net /CTRL_TXD: track 50.6 -> 33.9 mm, vias 2 -> 1
- net Net-(C9-Pad2): track 16.6 -> 32.9 mm, vias 0 -> 2
- net /FlickImp: track 91.6 -> 78.3 mm, vias 2 -> 4
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Other:
- board text added: "+"
- board text added: "-"
- board text added: "3V3"
- board text added: "5V"
- board text added: "In"
- board text added: "Synkino • Rev. C"
- board text added: "T"
- board text added: "^"
- board text removed: "Synkino • Rev. B"
